File: KiCAD-Source/ADS1115.kicad_sch (KiCad schematic)
At the start: 14 parts, among them J17 1x2-JSTXH, J18 1x2-JSTXH, J19 1x2-JSTXH, J20 1x2-JSTXH, U3 ADS1115IDGSR

Commit message: Added titleblocks to drawings
Other:
- company: (none) -> Pera @ https://transfur.science/f191
- title: (none) -> ThermEX26 Klipper Thermistor Expansion
Changed lines of the file:
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@@
 	(generator_version "9.0")
 	(paper "A5")
+	(title_block
+		(title "ThermEX26 Klipper Thermistor Expansion")
+		(date "2025-04-07")
+		(rev "2")
+		(company "Pera @ https://transfur.science/f191")
+		(comment 1 "CERN OHL v2 - S")
+		(comment 3 "https://github.com/comradef191/ThermEX")
+	)
 	(rectangle
 		(start 69.85 19.05)
