File: KiCAD-Source/ThermEX26.kicad_sch (KiCad schematic)
At the start: 22 parts, among them J1 2.54_1x5-M, J14 2.54_2x4-M, J15 1x4-JSTXH, J16 1x4-JSTXH, J2 2.54_2x5-M, J3 2.54_1x5-M, U2 TPS7A2033PDBVR

Commit message: Added titleblocks to drawings
Other:
- company: (none) -> Pera @ https://transfur.science/f191
- title: (none) -> ThermEX26 Klipper Thermistor Expansion
Changed lines of the file:
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@@
 	(generator_version "9.0")
 	(paper "A5")
+	(title_block
+		(title "ThermEX26 Klipper Thermistor Expansion")
+		(date "2025-04-07")
+		(rev "1")
+		(company "Pera @ https://transfur.science/f191")
+		(comment 1 "CERN OHL v2 - S")
+		(comment 3 "https://github.com/comradef191/ThermEX")
+	)
 	(rectangle
 		(start 175.26 43.815)
@@
 		)
 		(instances
-			(project "ThermEX10-Stack"
+			(project "ThermEX26"
 				(path "/31305e3c-4102-45f5-9b4f-137974626130"
 					(page "9")
@@
 		)
 		(instances
-			(project "ThermEX10-Stack"
+			(project "ThermEX26"
 				(path "/31305e3c-4102-45f5-9b4f-137974626130"
 					(page "3")
@@
 		)
 		(instances
-			(project "ThermEX10-Stack"
+			(project "ThermEX26"
 				(path "/31305e3c-4102-45f5-9b4f-137974626130"
 					(page "7")
@@
 		)
 		(instances
-			(project "ThermEX10-Stack"
+			(project "ThermEX26"
 				(path "/31305e3c-4102-45f5-9b4f-137974626130"
 					(page "4")
@@
 		)
 		(instances
-			(project "ThermEX10-Stack"
+			(project "ThermEX26"
 				(path "/31305e3c-4102-45f5-9b4f-137974626130"
 					(page "11")
@@
 		)
 		(instances
-			(project "ThermEX10-Stack"
+			(project "ThermEX26"
 				(path "/31305e3c-4102-45f5-9b4f-137974626130"
 					(page "15")
@@
 		)
 		(instances
-			(project "ThermEX10-Stack"
+			(project "ThermEX26"
 				(path "/31305e3c-4102-45f5-9b4f-137974626130"
 					(page "5")
@@
 		)
 		(instances
-			(project "ThermEX10-Stack"
+			(project "ThermEX26"
 				(path "/31305e3c-4102-45f5-9b4f-137974626130"
 					(page "12")
@@
 		)
 		(instances
-			(project "ThermEX10-Stack"
+			(project "ThermEX26"
 				(path "/31305e3c-4102-45f5-9b4f-137974626130"
 					(page "6")
@@
 		)
 		(instances
-			(project "ThermEX10-Stack"
+			(project "ThermEX26"
 				(path "/31305e3c-4102-45f5-9b4f-137974626130"
 					(page "13")
@@
 		)
 		(instances
-			(project "ThermEX10-Stack"
+			(project "ThermEX26"
 				(path "/31305e3c-4102-45f5-9b4f-137974626130"
 					(page "10")
@@
 		)
 		(instances
-			(project "ThermEX10-Stack"
+			(project "ThermEX26"
 				(path "/31305e3c-4102-45f5-9b4f-137974626130"
 					(page "8")
@@
 		)
 		(instances
-			(project "ThermEX10-Stack"
+			(project "ThermEX26"
 				(path "/31305e3c-4102-45f5-9b4f-137974626130"
 					(page "14")
@@
 		)
 		(instances
-			(project "ThermEX10-Stack"
+			(project "ThermEX26"
 				(path "/31305e3c-4102-45f5-9b4f-137974626130"
 					(page "2")
