File: KiCAD-Source/Thermistor.kicad_sch (KiCad schematic)
At the start: 3 parts, among them J12 1x2-JSTXH

Commit message: Added titleblocks to drawings
Other:
- company: (none) -> Pera @ https://transfur.science/f191
- title: (none) -> ThermEX26 Klipper Thermistor Expansion
Changed lines of the file:
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@@
 	(generator "eeschema")
 	(generator_version "9.0")
-	(paper "A4")
+	(paper "A5")
+	(title_block
+		(title "ThermEX26 Klipper Thermistor Expansion")
+		(date "2025-04-07")
+		(rev "2")
+		(company "Pera @ https://transfur.science/f191")
+		(comment 1 "CERN OHL v2 - S")
+		(comment 3 "https://github.com/comradef191/ThermEX")
+	)
 	(junction
 		(at 104.14 62.23)
