File: ThermEX-Simple/ThermEX-Simple.kicad_sch (KiCad schematic)
At the start: 0 parts

Commit message: Simple ThermEX
Parts:
- added H1, H2, H3, H4: MountingHole, CustomFootprints:M3 Mounting Hole ~ Classic - No Keepout, symbol Mechanical:MountingHole
- added J1, J3: 2.54_1x5-M, Connector_PinHeader_2.54mm:PinHeader_1x05_P2.54mm_Vertical, symbol Connector_Generic:Conn_01x05
- added J15: 2.54_2x2-M, Connector_PinHeader_2.54mm:PinHeader_2x02_P2.54mm_Vertical, symbol Connector_Generic:Conn_02x02_Odd_Even
- added J16, J4: 1x4-JSTXH, Connector_JST:JST_XH_B4B-XH-A_1x04_P2.50mm_Vertical, symbol Connector_Generic:Conn_01x04
- added J2: 2.54_2x5-M, Connector_PinHeader_2.54mm:PinHeader_2x05_P2.54mm_Vertical, symbol Connector_Generic:Conn_02x05_Odd_Even
- added U1: ~, CustomFootprints:Socketed MCU - STM32 BlackPill, symbol CustomSymbols:STM32F401_Black_Pill
Connections:
- new net +3V3: J16.1 (Pin_1), J3.1 (Pin_1), J3.2 (Pin_2), J3.3 (Pin_3), J3.4 (Pin_4), J3.5 (Pin_5), J4.1 (Pin_1), U1.18 (3V3)
- new net ADC-0: U1.6 (PA0)
- new net ADC-1: U1.7 (PA1)
- new net ADC-2: U1.8 (PA2)
- new net ADC-3: U1.9 (PA3)
- new net ADC-4: U1.10 (PA4)
- new net ADC-5: U1.11 (PA5)
- new net ADC-6: U1.12 (PA6)
- new net ADC-7: U1.13 (PA7)
- new net ADC-8: U1.14 (PB0)
- new net ADC-9: U1.15 (PB1)
- new net GND: J1.1 (Pin_1), J1.2 (Pin_2), J1.3 (Pin_3), J1.4 (Pin_4), J1.5 (Pin_5), J16.4 (Pin_4), J4.4 (Pin_4), U1.19 (GND), U1.39 (GND)
- new net GPIO-1: J2.9 (Pin_9), U1.2 (PC13)
- new net GPIO-10: J2.6 (Pin_6), U1.27 (PA10)
- new net GPIO-11: J2.5 (Pin_5), U1.26 (PA9)
- new net GPIO-12: J15.3 (Pin_3), U1.21 (PB12)
- new net GPIO-2: J2.7 (Pin_7), U1.3 (PC14)
- new net GPIO-3: J2.10 (Pin_10), U1.4 (PC15)
- new net GPIO-4: J2.8 (Pin_8), U1.16 (PB2)
- new net GPIO-5: J2.3 (Pin_3), U1.37 (PB9)
- new net GPIO-6: J2.1 (Pin_1), U1.36 (PB8)
- new net GPIO-8: J2.4 (Pin_4), U1.33 (PB5)
- new net GPIO-9: J2.2 (Pin_2), U1.30 (PA15)
- new net I2C-SCL-1: J16.3 (Pin_3), U1.34 (PB6)
- new net I2C-SCL-2: U1.17 (PB10)
- new net I2C-SCL-3: J4.3 (Pin_3), U1.25 (PA8)
- new net I2C-SDA-1: J16.2 (Pin_2), U1.35 (PB7)
- new net I2C-SDA-2: U1.31 (PB3)
- new net I2C-SDA-3: J4.2 (Pin_2), U1.32 (PB4)
- new net SPI2-MISO: J15.1 (Pin_1), U1.23 (PB14)
- new net SPI2-MOSI: J15.2 (Pin_2), U1.24 (PB15)
- new net SPI2-SCK: J15.4 (Pin_4), U1.22 (PB13)
- no-connect marks 0 -> 7
Other:
- added sheet Thermistor1 (Thermistor.kicad_sch)
- added sheet Thermistor10 (Thermistor.kicad_sch)
- added sheet Thermistor2 (Thermistor.kicad_sch)
- added sheet Thermistor3 (Thermistor.kicad_sch)
- added sheet Thermistor4 (Thermistor.kicad_sch)
- added sheet Thermistor5 (Thermistor.kicad_sch)
- added sheet Thermistor6 (Thermistor.kicad_sch)
- added sheet Thermistor7 (Thermistor.kicad_sch)
- added sheet Thermistor8 (Thermistor.kicad_sch)
- added sheet Thermistor9 (Thermistor.kicad_sch)
- note added: "Extra GPIO Breakout"
- note added: "M3 Bolts"
- note added: "On-Board ADCs; Extra Thermistors"
- note added: "STM32F401 Blackpill"
