File: ThermEX10-S/ThermEX-Simple.kicad_sch (KiCad schematic)
At the start: 11 parts, among them J1 2.54_1x5-M, J15 2.54_2x2-M, J16 1x4-JSTXH, J2 2.54_2x5-M, J3 2.54_1x5-M, J4 1x4-JSTXH

Commit message: Quick Fix
Parts:
- U1: value ~ -> STM32F401 Blackpill
Changed lines of the file:
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@@
 			)
 		)
-		(property "Value" "~"
+		(property "Value" "STM32F401 Blackpill"
 			(at 25.4 8.89 0)
 			(effects
