File: ThermEX10-S/Thermistor.kicad_sch (KiCad schematic)
At the start: 3 parts, among them J5 1x2-JSTXH

Commit message: Quick Fix
Parts:
- C1: LCSC C14663 -> (none)
- J5: LCSC C5160911 -> (none)
- R1: LCSC C2989672 -> (none)
Changed lines of the file:
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@@
-			)
-		)
-		(property "LCSC" " C14663"
-			(at 113.03 63.5 0)
-			(effects
-				(font
-					(size 1.27 1.27)
-				)
-				(hide yes)
 			)
 		)
@@
 			)
 		)
-		(property "LCSC" "C5160911"
-			(at 121.92 66.04 0)
-			(effects
-				(font
-					(size 1.27 1.27)
-				)
-				(hide yes)
-			)
-		)
 		(pin "1"
 		)
@@
 			(at 113.03 73.66 0)
 			(effects
-				(font
-					(size 1.27 1.27)
-				)
-				(hide yes)
-			)
-		)
-		(property "LCSC" "C2989672"
-			(at 113.03 73.66 0)
-			(effects
